File: DMH_Dual_VCA_Mk3_PCB_Controls/Controls.kicad_sch (KiCad schematic)
At the start: 21 parts, among them SW2 SW_DPDT_3way, U8 TL074

Commit message: Schematic labeling in progress
Parts:
- added R59, R60, R61, R62, R63, R64: 100k, Resistor_THT:R_Axial_DIN0207_L6.3mm_D2.5mm_P7.62mm_Horizontal, symbol Device:R_US
Connections:
- net CV Att A1: no longer names the net of RV7.2, RV7.3, U8.1
- net CV Att A1: now also R59.1
- net CV Att A2: no longer names the net of RV11.2, RV11.3, U8.8
- net CV Att A2: now also R60.1
- net CV Att B1: no longer names the net of RV8.2, RV8.3, U8.7
- net CV Att B1: now also R61.1
- net CV Att B2: no longer names the net of RV12.2, RV12.3, U8.14
- net CV Att B2: now also R62.1
- net Offset pot A: no longer names the net of RV13.2
- net Offset pot A: now also R63.1
- net Offset pot B: no longer names the net of RV14.2
- net Offset pot B: now also R64.1
- new net Processed_CV_A: R59.2, R60.2, R63.2
- new net Processed_CV_B: R61.2, R62.2, R64.2
Other:
- moved on the sheet: C3, C4, R4, R52, R53, R54, R55, RV10, RV11, RV12, RV13, RV14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
