File: DMH_Dual_VCA_Mk3_PCB_Controls/Controls.kicad_sch (KiCad schematic)
At the start: 27 parts, among them SW1 SW_DPDT_3way, U9 TL074

Commit message: Fixed Alps RK09L pot 3D model
Parts:
- RV6: footprint Potentiometer_THT:Potentiometer_Alps_RK09L_Double_Vertical -> SynthStuff:Potentiometer_Alps_RK09L_Double_Vertical
Changed lines of the file:
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@@
 			)
 		)
-		(property "Footprint" "Potentiometer_THT:Potentiometer_Alps_RK09L_Double_Vertical"
+		(property "Footprint" "SynthStuff:Potentiometer_Alps_RK09L_Double_Vertical"
 			(at 31.75 177.8 0)
 			(hide yes)
@@
 			)
 		)
-		(property "Footprint" "Potentiometer_THT:Potentiometer_Alps_RK09L_Double_Vertical"
+		(property "Footprint" "SynthStuff:Potentiometer_Alps_RK09L_Double_Vertical"
 			(at 82.55 177.8 0)
 			(hide yes)
