File: DMH_Dual_VCA_Mk3_PCB_Controls/DMH_Dual_VCA_Mk3_PCB_Controls.kicad_sch (KiCad schematic)
At the start: 1 part, among them J11 Conn_01x04_PinHeader

Commit message: Restarting schematic drawing
Parts:
- removed J11: Conn_01x04_PinHeader, Connector_PinSocket_2.54mm:PinSocket_1x04_P2.54mm_Vertical, symbol SynthStuff:Conn_01x04_PinHeader
- added J1, J2, J3, J4, J5, J6, J7, J8, J9: TRS_Jack_6.35mm_Sw, SynthStuff:CUI_SJ-63083D, symbol SynthStuff:TRS_Jack_6.35mm_Sw
- added R1, R4: 33k, Resistor_THT:R_Axial_DIN0207_L6.3mm_D2.5mm_P7.62mm_Horizontal, symbol Device:R_US
- added RV1: 100k, SynthStuff:Potentiometer_TT_P110KH1, symbol Device:R_Potentiometer_US
- added RV10, RV9: 50k, Potentiometer_THT:Potentiometer_Bourns_3296W_Vertical, symbol Device:R_Potentiometer_Trim_US
- added U1: TL074, Package_DIP:DIP-14_W7.62mm_Socket, symbol Amplifier_Operational:TL074
Connections:
- new net: RV1.2, U1.3 (+)
- new net: R1.1, RV1.3
- new net: R1.2, RV9.1, U1.2 (-)
- new net: RV9.2, RV9.3, U1.1
- new net: R4.2, RV10.1, U1.6 (-)
- new net: RV10.2, RV10.3, U1.7
- new net GND: RV1.1
Other:
- removed sheet 2nd VCA
- removed sheet Clipping
- removed sheet Inputs and Outputs
- removed sheet Main VCA A
- removed sheet Main VCA B
- added sheet VCA_DiffAmp_Subcircuit (VCA_DiffAmp_Subcircuit.kicad_sch)

Commit message: Experimenting with VCA design blocks
Connections:
- net at RV1.3: no longer R1.1
- net at R1.2, U1.2 (-): no longer RV9.1
- net at RV9.2, U1.1: no longer RV9.3
- net at R4.2, U1.6 (-): no longer RV10.1
- net at RV10.2, U1.7: no longer RV10.3
Other:
- removed sheet VCA_DiffAmp_Subcircuit
- added sheet VCA_1 (VCA_DiffAmp_SM_H.kicad_sch)
- added sheet VCA_2 (VCA_DiffAmp_SM_H.kicad_sch)
- added sheet VCA_3 (VCA_DiffAmp_SM_H.kicad_sch)
- added sheet VCA_4 (VCA_DiffAmp_SM_H.kicad_sch)

Commit message: Redesigned schematic layout
Parts:
- removed R1, R4: 33k, Resistor_THT:R_Axial_DIN0207_L6.3mm_D2.5mm_P7.62mm_Horizontal, symbol Device:R_US
- removed RV1: 100k, SynthStuff:Potentiometer_TT_P110KH1, symbol Device:R_Potentiometer_US
- removed RV10, RV9: 50k, Potentiometer_THT:Potentiometer_Bourns_3296W_Vertical, symbol Device:R_Potentiometer_Trim_US
- removed U1: TL074, Package_DIP:DIP-14_W7.62mm_Socket, symbol Amplifier_Operational:TL074
- added C1, C2: 47uF, Capacitor_THT:CP_Radial_D5.0mm_P2.00mm, symbol Device:C_Polarized
- added C10, C33, C34, C35, C36, C9: 100nF, Capacitor_THT:C_Disc_D4.3mm_W1.9mm_P5.00mm, symbol Device:C
- added C12: 22pF, Capacitor_THT:C_Disc_D3.0mm_W2.0mm_P2.50mm, symbol Device:C
- added D1, D2: SB140, Diode_THT:D_DO-41_SOD81_P10.16mm_Horizontal, symbol Diode:SB140
- added D3, D4: 1N4148, Diode_THT:D_DO-35_SOD27_P7.62mm_Horizontal, symbol Diode:1N4148
- added J100: IDC_02x05, SynthStuff:IDC-Header_2x05_P2.54mm_Vertical_Eurorack, symbol SynthStuff:Eurorack_Power_Connector_10Pin
- added J14: Conn_01x01, Connector_PinHeader_2.54mm:PinHeader_1x01_P2.54mm_Vertical, symbol Connector_Generic:Conn_01x01
- added J15: Conn_01x06, Connector_PinSocket_2.54mm:PinSocket_1x06_P2.54mm_Vertical, symbol Connector_Generic:Conn_01x06
- added J16: Conn_01x06, Connector_PinHeader_2.54mm:PinHeader_1x06_P2.54mm_Vertical, symbol Connector_Generic:Conn_01x06
- added J200: IDC_02x05, SynthStuff:IDC-Header_2x05_P2.54mm_Vertical_BackBone, symbol SynthStuff:BackBone_Connector_10Pin
- added JP1: Jumper, symbol Jumper:Jumper_3_Bridged12
- added R2, R73: 3k3, Resistor_THT:R_Axial_DIN0207_L6.3mm_D2.5mm_P7.62mm_Horizontal, symbol Device:R_US
- added R59, R60, R61, R62, R63, R64, R65, R66, R69, R70, R71, R72, R74, R75, R76: 100k, Resistor_THT:R_Axial_DIN0207_L6.3mm_D2.5mm_P7.62mm_Horizontal, symbol Device:R_US
- added R68: 33k, Resistor_THT:R_Axial_DIN0207_L6.3mm_D2.5mm_P7.62mm_Horizontal, symbol Device:R_US
- added R77, R78: 20k, Resistor_THT:R_Axial_DIN0207_L6.3mm_D2.5mm_P7.62mm_Horizontal, symbol Device:R_US
- added R79: 10k, Resistor_THT:R_Axial_DIN0207_L6.3mm_D2.5mm_P7.62mm_Horizontal, symbol Device:R_US
- added RV16: 50k, Potentiometer_THT:Potentiometer_Bourns_3296W_Vertical, symbol Device:R_Potentiometer_Trim_US
- added U10: TL072, Package_DIP:DIP-8_W7.62mm_Socket, symbol Amplifier_Operational:TL072
- added U11: TL074, Package_DIP:DIP-14_W7.62mm_Socket, symbol Amplifier_Operational:TL074
- added U5, U6: LM4040LP-5, Package_TO_SOT_THT:TO-92_Inline, symbol Reference_Voltage:LM4040LP-5
Connections:
- net GND: now also J1.S (1), J2.S (1), J3.S (1), J4.S (1), J5.S (1), J6.S (1), J7.S (1), J8.S (1), J9.S (1), C1.2, C10.2, C2.1, C33.2, C34.1, C35.2, C36.1, C9.2, J100.2a (Pin_2a), J100.2b (Pin_2b), J100.3a (Pin_3a), J100.3b (Pin_3b), J100.4a (Pin_4a), J100.4b (Pin_4b), J14.1 (Pin_1), J200.5 (Pin_5), R76.2, U10.5 (+), U11.10 (+), U11.12 (+), U5.3 (A), U6.2 (K)
- net VCA_A_Tier1/CV_Mix_In: now also R59.2, R60.2, R61.2
- net VCA_A_Tier2/CV_Mix_In: now also R65.2, R71.2
- net VCA_B_Tier1/CV_Mix_In: now also R62.2, R63.2, R64.2
- net VCA_B_Tier2/CV_Mix_In: now also R66.2, R72.2
- net Output A: now reaches J4.T (3)
- net Output A N: now reaches J4.TN (2)
- net Output A N: now also J200.2 (Pin_2)
- net Input B: now reaches J5.T (3)
- net Input B N: now reaches J5.TN (2)
- net Input B N: now also J200.9 (Pin_9)
- net Output B: now reaches J8.T (3)
- net Output B N: now reaches J8.TN (2)
- net Output B N: now also J200.8 (Pin_8)
- net CV In A1: now reaches J2.T (3)
- net CV In A1 N: now reaches J2.TN (2)
- net CV In A1 N: now also J200.3 (Pin_3)
- net CV In A2: now reaches J3.T (3)
- net CV In A2 N: now reaches J3.TN (2)
- net CV In A2 N: now also J200.4 (Pin_4)
- net CV In PT: now reaches J9.T (3)
- net CV In PT: now also R68.1
- net CV In PT N: now reaches J9.TN (2)
- net CV In PT N: now also JP1.2 (C)
- net Input A: now reaches J1.T (3)
- net Input A N: now reaches J1.TN (2)
- net Input A N: now also J200.1 (Pin_1)
- net CV In B1: now reaches J6.T (3)
- net CV In B1 N: now reaches J6.TN (2)
- net CV In B1 N: now also J200.7 (Pin_7)
- net CV In B2: now reaches J7.T (3)
- net CV In B2 N: now reaches J7.TN (2)
- net CV In B2 N: now also J200.6 (Pin_6)
- new net: R77.1, R78.2, R79.2, U11.9 (-)
- new net: C12.1, D3.1 (K), D4.2 (A), U11.1
- new net: C12.2, D3.2 (A), R74.2, U11.2 (-)
- new net: U11.13 (-), U11.14
- new net: J200.10 (Pin_10), JP1.1 (A)
- new net: R68.2, RV16.1, U10.2 (-)
- new net: D2.1 (K), J100.1a (Pin_1a), J100.1b (Pin_1b)
- new net: D1.2 (A), J100.5a (Pin_5a), J100.5b (Pin_5b)
- new net: D4.1 (K), R76.1, U11.5 (+)
- new net: R69.2, R70.1, U10.6 (-)
- new net: R75.1, R77.2, U11.7
- new net: R74.1, R75.2, U11.6 (-)
- new net +12V: C1.1, C33.1, C35.1, D1.1 (K), R2.2, R73.2, U10.8 (V+), U11.4 (V+)
- new net +5V: C9.1, JP1.3 (B), R73.1, U5.2 (K)
- new net -12V: C2.2, C34.2, C36.2, D2.2 (A), U10.4 (V-), U11.11 (V-)
- new net -5V: C10.1, R2.1, R79.1, U6.3 (A)
- new net Attenuverted CV PT: R66.1, R69.1, RV16.2, RV16.3, U10.1
- new net Balanced Offset: R78.1, U11.8
- new net CV PT Offset: R71.1, R72.1
- new net Controls/CV Att A1: R59.1
- new net Controls/CV Att A2: R60.1
- new net Controls/CV Att B1: R62.1
- new net Controls/CV Att B2: R63.1
- new net Controls/CV PT Pot G1: U10.3 (+)
- new net Controls/CV PT Pot G2: U11.3 (+)
- new net Controls/Offset pot A: R61.1
- new net Controls/Offset pot B: R64.1
- new net Inverted CV PT: R70.2, U10.7
- new net Processed CV PT: R65.1
- no-connect marks 0 -> 18
Other:
- sheet VCA_1 renamed VCA_A_Tier1
- sheet VCA_2 renamed VCA_A_Tier2
- sheet VCA_3 renamed VCA_B_Tier1
- sheet VCA_4 renamed VCA_B_Tier2
- removed sheet Power
- added sheet Clipping (Clipping.kicad_sch)
- added sheet Controls (Controls.kicad_sch)

Commit message: schematic labeling in progress
Connections:
- net Attenuverted CV PT renamed Attenuverted_CV_PT_m
- net Attenuverted_CV_PT_m: no longer R66.1
- net Balanced Offset renamed Balanced_Offset_m
- net CV In A1 renamed CV_In_A1_m
- net CV In A1 N renamed CV_In_A1_N_m
- net CV In A2 renamed CV_In_A2_m
- net CV In A2 N renamed CV_In_A2_N_m
- net CV In B1 renamed CV_In_B1_m
- net CV In B1 N renamed CV_In_B1_N_m
- net CV In B2 renamed CV_In_B2_m
- net CV In B2 N renamed CV_In_B2_N_m
- net CV In PT renamed CV_In_PT
- net CV_In_PT: no longer J9.T (3)
- net CV In PT N renamed CV_In_PT_N_m
- net CV PT Offset renamed CV_PT_Offset
- net Controls/CV PT Pot G1 renamed CV_PT_Pot_G1_m
- net Controls/CV PT Pot G2 renamed CV_PT_Pot_G2_m
- net Input A renamed Input_A_m
- net Input A N renamed Input_A_N_m
- net Input_A_N_m: no longer J1.TN (2)
- net Input B renamed Input_B_m
- net Input B N renamed Input_B_N_m
- net Inverted CV PT renamed Inverted_CV_PT_m
- net Output A renamed Output_A_m
- net Output A N renamed Output_A_N_m
- net Output B renamed Output_B_m
- net Output B N renamed Output_B_N_m
- net Processed CV PT renamed Processed_CV_PT
- new net Attenuverted_CV_PT: R66.1
- new net CV_In_PT_m: J9.T (3)
- new net Input_A_N_m_m: J1.TN (2)
Other:
- moved on the sheet: R65, R66, R68, R69, R70, R71, R72, RV16, U10A, U10B

Commit message: Schematic labeling in progress
Parts:
- removed R59, R60, R61, R62, R63, R64: 100k, Resistor_THT:R_Axial_DIN0207_L6.3mm_D2.5mm_P7.62mm_Horizontal, symbol Device:R_US
- added J17: Conn_01x08, Connector_PinSocket_2.54mm:PinSocket_1x06_P2.54mm_Vertical, symbol Connector_Generic:Conn_01x08
- added J18: Conn_01x08, Connector_PinHeader_2.54mm:PinHeader_1x06_P2.54mm_Vertical, symbol Connector_Generic:Conn_01x08
- added J19, J20, J21, J22: Conn_02x03_Odd_Even, Connector_PinHeader_2.54mm:PinHeader_2x03_P2.54mm_Horizontal, symbol Connector_Generic:Conn_02x03_Odd_Even
- added J23, J24: Conn_01x06, Connector_PinHeader_2.54mm:PinHeader_1x06_P2.54mm_Vertical, symbol Connector_Generic:Conn_01x06
Connections:
- net Attenuverted_CV_PT is gone; now on net Attenuverted_CV_PT_m: R66.1
- net CV_In_PT is gone; now on net CV_In_PT_m: R68.1
- net +12V: now also J19.1 (Pin_1), J20.1 (Pin_1), J21.1 (Pin_1), J22.1 (Pin_1), J23.2 (Pin_2), J24.2 (Pin_2)
- net +5V: now also J23.4 (Pin_4), J24.4 (Pin_4)
- net -12V: now also J19.3 (Pin_3), J20.3 (Pin_3), J21.3 (Pin_3), J22.3 (Pin_3), J23.3 (Pin_3), J24.3 (Pin_3)
- net -5V: now also J23.5 (Pin_5), J24.5 (Pin_5)
- net Attenuverted_CV_PT_c: now also J18.3 (Pin_3)
- net Balanced_Offset_c: now also J18.1 (Pin_1)
- net Balanced_Offset_m: now also J17.1 (Pin_1)
- net CV_In_A1_c: now also J16.3 (Pin_3)
- net CV_In_A1_m: now also J15.3 (Pin_3)
- net CV_In_A2_c: now also J16.4 (Pin_4)
- net CV_In_A2_m: now also J15.4 (Pin_4)
- net CV_In_B1_c: now also J16.5 (Pin_5)
- net CV_In_B1_m: now also J15.5 (Pin_5)
- net CV_In_B2_c: now also J16.6 (Pin_6)
- net CV_In_B2_m: now also J15.6 (Pin_6)
- net CV_In_PT_c: now also J18.8 (Pin_8)
- net CV_In_PT_m: now also J17.8 (Pin_8)
- net CV_PT_Offset_c: now also J18.5 (Pin_5)
- net CV_PT_Pot_G1_c: now also J18.6 (Pin_6)
- net CV_PT_Pot_G1_m: now also J17.6 (Pin_6)
- net CV_PT_Pot_G2_c: now also J18.7 (Pin_7)
- net CV_PT_Pot_G2_m: now also J17.7 (Pin_7)
- net GND: now also J19.5 (Pin_5), J20.5 (Pin_5), J21.5 (Pin_5), J22.5 (Pin_5), J23.1 (Pin_1), J23.6 (Pin_6), J24.1 (Pin_1), J24.6 (Pin_6)
- net Inverted_CV_PT_c: now also J18.2 (Pin_2)
- net Processed_CV_PT_c: now also J18.4 (Pin_4)
- net Processed_mV_A_m: now reaches J15.1 (Pin_1)
- net Processed_mV_B_m: now reaches J15.2 (Pin_2)
- net Processed_CV_A_c: now reaches J16.1 (Pin_1)
- net Processed_CV_B_c: now reaches J16.2 (Pin_2)
- net CV_PT_Offset renamed CV_PT_Offset_m
- net CV_PT_Offset_m: now also J17.5 (Pin_5)
- net Processed_CV_PT renamed Processed_CV_PT_m
- net VCA_A_Tier2/CV_Mix_In renamed VCA_A_T2_CV_m
- net VCA_A_T2_CV_m: now also J21.2 (Pin_2)
- net VCA_B_Tier2/CV_Mix_In renamed VCA_B_T2_CV_m
- net VCA_B_T2_CV_m: now also J22.2 (Pin_2)
- new net Attenuverted_mV_PT_m: J17.3 (Pin_3)
- new net Inverted_mV_PT_m: J17.2 (Pin_2)
- new net Processed_mV_PT_m: J17.4 (Pin_4)
- new net VCA_A_T1_CV_m: J19.2 (Pin_2)
- new net VCA_A_T1_In_m: J19.4 (Pin_4)
- new net VCA_A_T1_Out_m: J19.6 (Pin_6)
- new net VCA_A_T2_In_m: J21.4 (Pin_4)
- new net VCA_A_T2_Out_m: J21.6 (Pin_6)
- new net VCA_B_T1_CV_m: J20.2 (Pin_2)
- new net VCA_B_T1_In_m: J20.4 (Pin_4)
- new net VCA_B_T1_Out_m: J20.6 (Pin_6)
- new net VCA_B_T2_In_m: J22.4 (Pin_4)
- new net VCA_B_T2_Out_m: J22.6 (Pin_6)
Other:
- sheet Controls ports: added Processed_CV_A, Processed_CV_B; removed CV Att A1, CV Att A2, CV Att B1, CV Att B2, Offset pot A, Offset pot B
- moved on the sheet: C12, D3, D4, J15, J16, R65, R66, R68, R69, R70, R71, R72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
