File: DMH_Dual_VCA_Mk3_PCB_Main/Clipping.kicad_sch (KiCad schematic)
At the start: 50 parts, among them J21 Conn_01x08, J24 Conn_01x08, Q10 BC548, Q11 BC548, Q12 BC548, Q9 BC548, SW2 SW_DPDT_OnOffOn_x2, U10 TL074

Commit message: Generated schematic and BoM
Other:
- title: (none) -> 074-2 Dual VCA Mk3
Changed lines of the file:
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@@
 	(paper "A4" portrait)
 	(title_block
+		(title "074-2 Dual VCA Mk3")
 		(company "DMH Instruments")
 		(comment 1 "PCB for 5 cm Kosmo format synthesizer module")
