File: DMH_Dual_VCA_Mk3_PCB_Main/DMH_Dual_VCA_Mk3_PCB_Main.kicad_pcb (KiCad board)
At the start: 2 copper layers, 49 x 175 mm, 98 parts, among them J1 TRS_Jack_6.35mm_Sw, J100 IDC_02x05, J11 Conn_01x06, J12 Conn_01x08, J13 Conn_01x06, J18 Conn_02x03_Odd_Even, J19 Conn_02x03_Odd_Even, J2 TRS_Jack_6.35mm_Sw, J20 Conn_01x01, J200 IDC_02x05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

Commit message: Main PCB routing in progress
Parts:
- moved C4 1.00 mm to (59.0, 50.5)
Connections:
- J200 pad 4: /Output_B_N_m -> /Output_A_N_m
- J200 pad 9: /Output_A_N_m -> /Output_B_N_m
Routing:
- net -12V: track 9.98 -> 263.9 mm
- net +12V: track 50.8 -> 261.6 mm
- net +5V: track 0.00 -> 164.1 mm
- net /Clipping/LED_B_pK_m: track 0.00 -> 115.7 mm
- net /Clip_Out_B_m: track 0.00 -> 109.5 mm
- net /Clip_Out_A_m: track 0.00 -> 107.3 mm
- net /CV_In_PT_m: track 0.00 -> 103.2 mm
- net Net-(U10C--): track 0.00 -> 86.9 mm
- net /VCA_A_Tier1/Signal_Out: track 0.00 -> 86.5 mm
- net /Attenuverted_CV_PT_m: track 0.00 -> 81.5 mm
- net Net-(U10B--): track 0.00 -> 80.6 mm
- net /Balanced_Offset_m: track 0.00 -> 79.7 mm
- net /Clipping/LED_B_pA_m: track 0.00 -> 75.5 mm
- net /Inverted_CV_PT_m: track 0.00 -> 74.2 mm
- net /Clipping/Clip_Sw_p1_m: track 0.00 -> 72.1 mm
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
Commit message: Main PCB routing done
Parts:
- moved D11 0.80 mm to (96.5, 124.0)
- moved D12 0.80 mm to (96.5, 129.8)
- moved Q9 0.61 mm to (88.3, 62.2)
- moved D1 0.20 mm to (77.1, 83.2)
Connections:
- JP3 pad 1: Net-(J200-Pin_3) -> Net-(J200-Pin_2)
- JP4 pad 1: Net-(J200-Pin_2) -> Net-(J200-Pin_3)
Routing:
- net /CV_PT_Pot_G2_m: track 0.00 -> 138.0 mm
- net /Input_B_m: track 0.00 -> 132.1 mm
- net /Clipping/Clip_Sw_p4_m: track 14.8 -> 112.3 mm, vias 0 -> 3
- net /CV_In_B1_m: track 0.00 -> 81.4 mm
- net /CV_In_B1_N_m: track 0.00 -> 61.6 mm
- net /Input_B_N_m: track 0.00 -> 59.6 mm
- net /CV_In_A2_N_m: track 0.00 -> 58.7 mm
- net /Input_A_N_m: track 0.00 -> 51.2 mm
- net /CV_In_A1_m: track 15.1 -> 53.1 mm
- net /CV_In_B2_m: track 0.00 -> 26.5 mm
- net /Balanced_Offset_m: track 79.7 -> 94.6 mm
- net /Attenuverted_CV_PT_m: track 81.5 -> 94.1 mm
- net /Input_A_m: track 65.9 -> 74.9 mm
- net Net-(J200-Pin_2): track 23.0 -> 14.2 mm
- net Net-(R100-Pad1): track 47.5 -> 55.1 mm
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