File: DMH_Dual_VCA_Mk3_PCB_Main/DMH_Dual_VCA_Mk3_PCB_Main.kicad_sch (KiCad schematic)
At the start: 59 parts, among them J1 TRS_Jack_6.35mm_Sw, J100 IDC_02x05, J11 Conn_01x06, J12 Conn_01x08, J13 Conn_01x06, J14 Conn_01x06, J15 Conn_01x08, J16 Conn_01x06, J18 Conn_02x03_Odd_Even, J19 Conn_02x03_Odd_Even, J2 TRS_Jack_6.35mm_Sw, J20 Conn_01x01, J200 IDC_02x05, J22 Conn_02x03_Odd_Even, J23 Conn_02x03_Odd_Even, J3 TRS_Jack_6.35mm_Sw, J4 TRS_Jack_6.35mm_Sw, J5 TRS_Jack_6.35mm_Sw, J6 TRS_Jack_6.35mm_Sw, J7 TRS_Jack_6.35mm_Sw, J8 TRS_Jack_6.35mm_Sw, J9 TRS_Jack_6.35mm_Sw, U1 LM4040LP-5, U2 LM4040LP-5, U3 TL074, U4 TL072

Commit message: Generated schematic and BoM
Other:
- title: (none) -> 074-2 Dual VCA Mk3
Changed lines of the file:
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@@
 	(paper "A3")
 	(title_block
+		(title "074-2 Dual VCA Mk3")
 		(rev "1")
 		(company "DMH Instruments")
