File: DMH_Dual_VCA_Mk3_PCB_Main/VCA_DiffAmp_SM_H.kicad_sch (KiCad schematic)
At the start: 19 parts, among them J25 Conn_02x03_Odd_Even, Q1 BC548, Q2 BC548, U5 TL072

Commit message: Generated schematic and BoM
Other:
- title: (none) -> 074-2 Dual VCA Mk3
Changed lines of the file:
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@@
 	(paper "A4")
 	(title_block
+		(title "074-2 Dual VCA Mk3")
 		(company "DMH Instruments")
 		(comment 1 "PCB for 5 cm Kosmo format synthesizer module")
