File: DMH_Dual_VCA_Mk3_PANEL/DMH_Dual_VCA_Mk3_PANEL.kicad_pcb (KiCad board)
At the start: 2 copper layers, 50 x 200 mm, 25 parts, among them J0 Panel_GND_Solder_Wire_Pad

Commit message: Changed pan pot panel hole to match Alps RK09L pot
Parts:
- H20: footprint SynthStuff:Pot_Cutout_Tiny_attv_RD901F -> SynthStuff:Pot_Cutout_Tiny_attv_RK09L
- moved J0 10.0 mm to (55.0, 104.0)
Other:
- board text added: "Mk3.1 - June 2026"
- board text removed: "Mk3.0 - June 2026"
Changed lines of the file:
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@@
 		)
 	)
-	(footprint "SynthStuff:Pot_Cutout_Tiny_attv_RD901F"
+	(footprint "SynthStuff:Pot_Cutout_Tiny_attv_RK09L"
 		(layer "F.Cu")
 		(at 87.25 103.25)
@@
 		(sheetname "/")
 		(sheetfile "DMH_Dual_VCA_Mk3_PANEL.kicad_sch")
+		(units
+			(unit
+				(name "A")
+				(pins "1")
+			)
+		)
 		(attr through_hole)
 		(duplicate_pad_numbers_are_jumpers no)
@@
 		(fp_circle
 			(center 0 0)
-			(end 3.5 0)
+			(end 4.6 0)
 			(stroke
 				(width 0.05)
-				(type default)
+				(type solid)
 			)
 			(fill no)
@@
 		(pad "1" connect circle
 			(at 0 0)
-			(size 12 12)
+			(size 14 14)
 			(layers "F.Cu" "F.Mask")
 			(net "GND")
@@
 		(pad "1" connect circle
 			(at 0 0)
-			(size 12 12)
+			(size 14 14)
 			(layers "B.Cu" "B.Mask")
 			(net "GND")
@@
 	(footprint "SynthStuff:Panel_GND_SolderWirePad_5x10mm"
 		(layer "B.Cu")
-		(at 55 114 180)
+		(at 55 104 180)
 		(descr "Wire Pad, Square, SMD Pad,  5mm x 10mm,")
 		(tags "MesurementPoint Square SMDPad 5mmx10mm ")
@@
 		)
 	)
-	(gr_text "Mk3.0 - June 2026"
+	(gr_text "Mk3.1 - June 2026"
 		(at 75 222.95 0)
 		(layer "B.SilkS")
