File: DMH_Dual_VCA_Mk3_PANEL/DMH_Dual_VCA_Mk3_PANEL.kicad_sch (KiCad schematic)
At the start: 25 parts, among them J0 Panel_GND_Solder_Wire_Pad

Commit message: Changed pan pot panel hole to match Alps RK09L pot
Parts:
- H20: footprint SynthStuff:Pot_Cutout_Tiny_attv_RD901F -> SynthStuff:Pot_Cutout_Tiny_attv_RK09L
Changed lines of the file:
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@@
 			)
 		)
-		(property "Footprint" "SynthStuff:Pot_Cutout_Tiny_attv_RD901F"
+		(property "Footprint" "SynthStuff:Pot_Cutout_Tiny_attv_RK09L"
 			(at 127 153.67 0)
 			(hide yes)
